Commit message: renamed package, removed vendoring and updated installation

File: assets/g1/g1_29dof_with_hand_rev_1_0_ros.urdf (robot description, URDF)
Before this commit: robot g1_29dof_with_hand_rev_1_0, 54 links, 53 joints
Links:
- link head_link: geometry collision mesh filename=package://g1_pilot/assets/g1/meshes/head_link.STL; visual mesh filename=package://g1_pilot/assets/g1/meshes/head_link.STL
- link left_ankle_pitch_link: geometry collision mesh filename=package://g1_pilot/assets/g1/meshes/left_ankle_pitch_link.S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; visual mesh filename=package://g1_pilot/assets/g1/meshes/left_ankle_pitch_link.S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
- link left_ankle_roll_link: geometry collision sphere radius=0.005; collision sphere radius=0.005
- link left_elbow_link: geometry collision mesh filename=package://g1_pilot/assets/g1/meshes/left_elbow_link.STL; visual mesh filename=package://g1_pilot/assets/g1/meshes/left_elbow_link.STL
- link left_hand_index_0_link: geometry collision mesh filename=package://g1_pilot/assets/g1/meshes/left_hand_index_0_link.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; visual mesh filename=package://g1_pilot/assets/g1/meshes/left_hand_index_0_link.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
- link left_hand_index_1_link: geometry collision mesh filename=package://g1_pilot/assets/g1/meshes/left_hand_index_1_link.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; visual mesh filename=package://g1_pilot/assets/g1/meshes/left_hand_index_1_link.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
- link left_hand_middle_0_link: geometry collision mesh filename=package://g1_pilot/assets/g1/meshes/left_hand_middle_0_link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; visual mesh filename=package://g1_pilot/assets/g1/meshes/left_hand_middle_0_link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
- link left_hand_middle_1_link: geometry collision mesh filename=package://g1_pilot/assets/g1/meshes/left_hand_middle_1_link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; visual mesh filename=package://g1_pilot/assets/g1/meshes/left_hand_middle_1_link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
- link left_hand_palm_link: geometry collision mesh filename=package://g1_pilot/assets/g1/meshes/left_hand_palm_link.STL; visual mesh filename=package://g1_pilot/assets/g1/meshes/left_hand_palm_link.STL
- link left_hand_thumb_0_link: geometry collision mesh filename=package://g1_pilot/assets/g1/meshes/left_hand_thumb_0_link.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; visual mesh filename=package://g1_pilot/assets/g1/meshes/left_hand_thumb_0_link.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
- link left_hand_thumb_1_link: geometry collision box size=0.02 0.03 0.02; visual mesh filename=package://g1_pilot/assets/g1/meshes/left_hand_thumb_1_link.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
- link left_hand_thumb_2_link: geometry collision mesh filename=package://g1_pilot/assets/g1/meshes/left_hand_thumb_2_link.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; visual mesh filename=package://g1_pilot/assets/g1/meshes/left_hand_thumb_2_link.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
- link left_hip_pitch_link: geometry collision mesh filename=package://g1_pilot/assets/g1/meshes/left_hip_pitch_link.STL; visual mesh filename=package://g1_pilot/assets/g1/meshes/left_hip_pitch_link.STL
- link left_hip_roll_link: geometry collision mesh filename=package://g1_pilot/assets/g1/meshes/left_hip_roll_link.STL; visual mesh filename=package://g1_pilot/assets/g1/meshes/left_hip_roll_link.STL
- link left_hip_yaw_link: geometry collision mesh filename=package://g1_pilot/assets/g1/meshes/left_hip_yaw_link.STL; visual mesh filename=package://g1_pilot/assets/g1/meshes/left_hip_yaw_link.STL
- link left_knee_link: geometry collision mesh filename=package://g1_pilot/assets/g1/meshes/left_knee_link.STL; visual mesh filename=package://g1_pilot/assets/g1/meshes/left_knee_link.STL
- link left_shoulder_pitch_link: geometry collision cylinder length=0.05 radius=0.03; visual mesh filename=package://g1_pilot/assets/g1/meshes/left_shoulder_pitch_lin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
- link left_shoulder_roll_link: geometry collision cylinder length=0.03 radius=0.03; visual mesh filename=package://g1_pilot/assets/g1/meshes/left_shoulder_roll_link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
- link left_shoulder_yaw_link: geometry collision mesh filename=package://g1_pilot/assets/g1/meshes/left_shoulder_yaw_link.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; visual mesh filename=package://g1_pilot/assets/g1/meshes/left_shoulder_yaw_link.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
- link left_wrist_pitch_link: geometry collision mesh filename=package://g1_pilot/assets/g1/meshes/left_wrist_pitch_link.S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; visual mesh filename=package://g1_pilot/assets/g1/meshes/left_wrist_pitch_link.S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
- link left_wrist_roll_link: geometry collision mesh filename=package://g1_pilot/assets/g1/meshes/left_wrist_roll_link.STL; visual mesh filename=package://g1_pilot/assets/g1/meshes/left_wrist_roll_link.STL
- link left_wrist_yaw_link: geometry collision mesh filename=package://g1_pilot/assets/g1/meshes/left_wrist_yaw_link.STL; visual mesh filename=package://g1_pilot/assets/g1/meshes/left_wrist_yaw_link.STL
- link logo_link: geometry collision mesh filename=package://g1_pilot/assets/g1/meshes/logo_link.STL; visual mesh filename=package://g1_pilot/assets/g1/meshes/logo_link.STL
- link pelvis: geometry visual mesh filename=package://g1_pilot/assets/g1/meshes/pelvis.STL
- link pelvis_contour_link: geometry collision mesh filename=package://g1_pilot/assets/g1/meshes/pelvis_contour_link.STL; visual mesh filename=package://g1_pilot/assets/g1/meshes/pelvis_contour_link.STL
- link right_ankle_pitch_link: geometry collision mesh filename=package://g1_pilot/assets/g1/meshes/right_ankle_pitch_link.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; visual mesh filename=package://g1_pilot/assets/g1/meshes/right_ankle_pitch_link.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
- link right_ankle_roll_link: geometry collision sphere radius=0.005; collision sphere radius=0.005
- link right_elbow_link: geometry collision mesh filename=package://g1_pilot/assets/g1/meshes/right_elbow_link.STL; visual mesh filename=package://g1_pilot/assets/g1/meshes/right_elbow_link.STL
- link right_hand_index_0_link: geometry collision mesh filename=package://g1_pilot/assets/g1/meshes/right_hand_index_0_link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; visual mesh filename=package://g1_pilot/assets/g1/meshes/right_hand_index_0_link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
- link right_hand_index_1_link: geometry collision mesh filename=package://g1_pilot/assets/g1/meshes/right_hand_index_1_link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; visual mesh filename=package://g1_pilot/assets/g1/meshes/right_hand_index_1_link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
- link right_hand_middle_0_link: geometry collision mesh filename=package://g1_pilot/assets/g1/meshes/right_hand_middle_0_lin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; visual mesh filename=package://g1_pilot/assets/g1/meshes/right_hand_middle_0_lin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
- link right_hand_middle_1_link: geometry collision mesh filename=package://g1_pilot/assets/g1/meshes/right_hand_middle_1_lin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; visual mesh filename=package://g1_pilot/assets/g1/meshes/right_hand_middle_1_lin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
- link right_hand_palm_link: geometry collision mesh filename=package://g1_pilot/assets/g1/meshes/right_hand_palm_link.STL; visual mesh filename=package://g1_pilot/assets/g1/meshes/right_hand_palm_link.STL
- link right_hand_thumb_0_link: geometry collision mesh filename=package://g1_pilot/assets/g1/meshes/right_hand_thumb_0_link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; visual mesh filename=package://g1_pilot/assets/g1/meshes/right_hand_thumb_0_link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
- link right_hand_thumb_1_link: geometry collision box size=0.02 0.03 0.02; visual mesh filename=package://g1_pilot/assets/g1/meshes/right_hand_thumb_1_link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
- link right_hand_thumb_2_link: geometry collision mesh filename=package://g1_pilot/assets/g1/meshes/right_hand_thumb_2_link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; visual mesh filename=package://g1_pilot/assets/g1/meshes/right_hand_thumb_2_link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
- link right_hip_pitch_link: geometry collision mesh filename=package://g1_pilot/assets/g1/meshes/right_hip_pitch_link.STL; visual mesh filename=package://g1_pilot/assets/g1/meshes/right_hip_pitch_link.STL
- link right_hip_roll_link: geometry collision mesh filename=package://g1_pilot/assets/g1/meshes/right_hip_roll_link.STL; visual mesh filename=package://g1_pilot/assets/g1/meshes/right_hip_roll_link.STL
- link right_hip_yaw_link: geometry collision mesh filename=package://g1_pilot/assets/g1/meshes/right_hip_yaw_link.STL; visual mesh filename=package://g1_pilot/assets/g1/meshes/right_hip_yaw_link.STL
- link right_knee_link: geometry collision mesh filename=package://g1_pilot/assets/g1/meshes/right_knee_link.STL; visual mesh filename=package://g1_pilot/assets/g1/meshes/right_knee_link.STL
- link right_shoulder_pitch_link: geometry collision cylinder length=0.05 radius=0.03; visual mesh filename=package://g1_pilot/assets/g1/meshes/right_shoulder_pitch_li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
- link right_shoulder_roll_link: geometry collision cylinder length=0.03 radius=0.03; visual mesh filename=package://g1_pilot/assets/g1/meshes/right_shoulder_roll_lin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
- link right_shoulder_yaw_link: geometry collision mesh filename=package://g1_pilot/assets/g1/meshes/right_shoulder_yaw_link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; visual mesh filename=package://g1_pilot/assets/g1/meshes/right_shoulder_yaw_link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
- link right_wrist_pitch_link: geometry collision mesh filename=package://g1_pilot/assets/g1/meshes/right_wrist_pitch_link.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; visual mesh filename=package://g1_pilot/assets/g1/meshes/right_wrist_pitch_link.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
- link right_wrist_roll_link: geometry collision mesh filename=package://g1_pilot/assets/g1/meshes/right_wrist_roll_link.S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; visual mesh filename=package://g1_pilot/assets/g1/meshes/right_wrist_roll_link.S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
- link right_wrist_yaw_link: geometry collision mesh filename=package://g1_pilot/assets/g1/meshes/right_wrist_yaw_link.STL; visual mesh filename=package://g1_pilot/assets/g1/meshes/right_wrist_yaw_link.STL
- link torso_link: geometry collision mesh filename=package://g1_pilot/assets/g1/meshes/torso_link_rev_1_0.STL; visual mesh filename=package://g1_pilot/assets/g1/meshes/torso_link_rev_1_0.STL
- link waist_roll_link: geometry visual mesh filename=package://g1_pilot/assets/g1/meshes/waist_roll_link_rev_1_0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
- link waist_yaw_link: geometry visual mesh filename=package://g1_pilot/assets/g1/meshes/waist_yaw_link_rev_1_0.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

Commit message: changed urdf used for tf with standard names

File: assets/g1/g1_29dof_with_hand_rev_1_0_ros.urdf (robot description, URDF)
Before this commit: robot g1_29dof_with_hand_rev_1_0, 54 links, 53 joints
Links:
- removed link d435_link
- removed link g1_center
- removed link mid360_link
- added link base_link
- added link camera_link
- added link sensor
Joints:
- joint d435_joint: child d435_link -> camera_link
- joint g1_reference_to_pelvis_joint: parent g1_center -> base_link
- joint mid360_joint: child mid360_link -> torso_link; origin xyz=0.0002835 0.00003 0.41618 rpy=0 0.04014257279586953 0 -> xyz=-0.0002835 -0.00003 -0.41618 rpy=0 -0.04014257279586953 0; parent torso_link -> sensor

Commit message: reversing pelvis to torso link

File: assets/g1/g1_29dof_with_hand_rev_1_0_ros.urdf (robot description, URDF)
Before this commit: robot g1_29dof_with_hand_rev_1_0, 54 links, 53 joints
Joints:
- joint g1_reference_to_pelvis_joint: child pelvis -> base_link; parent base_link -> pelvis
- joint waist_pitch_joint: child torso_link -> waist_roll_link; parent waist_roll_link -> torso_link
- joint waist_roll_joint: child waist_roll_link -> waist_yaw_link; origin xyz=-0.0039635 0 0.044 rpy=0 0 0 -> xyz=0.0039635 0 -0.044 rpy=0 0 0; parent waist_yaw_link -> waist_roll_link
- joint waist_yaw_joint: child waist_yaw_link -> pelvis; parent pelvis -> waist_yaw_link

Commit message: revered joint direction for compatibility with a modified chain

File: assets/g1/g1_29dof_with_hand_rev_1_0_ros.urdf (robot description, URDF)
Before this commit: robot g1_29dof_with_hand_rev_1_0, 54 links, 53 joints
Joints:
- joint d435_joint: origin xyz=0.0799335 0.01753 0.41036 rpy=0 0.401426 0 -> xyz=0.0856235 0.03553 0.4407 rpy=0 0.501426 0
- joint waist_pitch_joint: axis 0 1 0 -> 0 -1 0
- joint waist_roll_joint: axis 1 0 0 -> -1 0 0
- joint waist_yaw_joint: axis 0 0 1 -> 0 0 -1

Commit message: camera robot calib, ik reset and updating goal topic

File: assets/g1/g1_29dof_with_hand_rev_1_0_ros.urdf (robot description, URDF)
Before this commit: robot g1_29dof_with_hand_rev_1_0, 54 links, 53 joints
Joints:
- joint d435_joint: origin xyz=0.0856235 0.03553 0.4407 rpy=0 0.501426 0 -> xyz=0.069560 0.019582 0.409726 rpy=0.023238 0.475734 0.001097

Commit message: eye base calibration

File: assets/g1/g1_29dof_with_hand_rev_1_0_ros.urdf (robot description, URDF)
Before this commit: robot g1_29dof_with_hand_rev_1_0, 54 links, 53 joints
Joints:
- joint d435_joint: origin xyz=0.069560 0.019582 0.409726 rpy=0.023238 0.475734 0.001097 -> xyz=0.068042 0.016300 0.414516 rpy=-0.111720 0.453641 0.026073

Commit message: eye base calib to perfection

File: assets/g1/g1_29dof_with_hand_rev_1_0_ros.urdf (robot description, URDF)
Before this commit: robot g1_29dof_with_hand_rev_1_0, 54 links, 53 joints
Joints:
- joint d435_joint: origin xyz=0.068042 0.016300 0.414516 rpy=-0.111720 0.453641 0.026073 -> xyz=0.068042 0.016300 0.414516 rpy=-0.011720 0.453641 0.026073
