Commit message: new camera mount transform

File: assets/g1/g1_29dof_with_hand_rev_1_0.urdf (robot description, URDF)
Before this commit: robot g1_29dof_with_hand_rev_1_0, 54 links, 53 joints
Joints:
- joint d435_joint: origin xyz=0.0576235 0.01753 0.42987 rpy=0 0.8307767239493009 0 -> xyz=0.0799335 0.01753 0.41036 rpy=0 0.401426 0

File: assets/g1/g1_29dof_with_hand_rev_1_0_ros.urdf (robot description, URDF)
Before this commit: robot g1_29dof_with_hand_rev_1_0, 54 links, 53 joints
Joints:
- joint d435_joint: origin xyz=0.0576235 0.01753 0.42987 rpy=0 0.8307767239493009 0 -> xyz=0.0799335 0.01753 0.41036 rpy=0 0.401426 0

Commit message: added practical limits to shoulder roll pitch and elbow joints

File: assets/g1/g1_29dof_with_hand_rev_1_0.urdf (robot description, URDF)
Before this commit: robot g1_29dof_with_hand_rev_1_0, 54 links, 53 joints
Joints:
- joint left_elbow_joint: limit lower=-1.0472 upper=2.0944 effort=25 velocity=37 -> lower=-0.7 upper=2.0944 effort=25 velocity=37
- joint left_shoulder_pitch_joint: limit lower=-3.0892 upper=2.6704 effort=25 velocity=37 -> lower=-1.3 upper=1.3 effort=25 velocity=37
- joint left_shoulder_roll_joint: limit lower=-1.5882 upper=2.2515 effort=25 velocity=37 -> lower=0.1 upper=1.59 effort=25 velocity=37
- joint right_elbow_joint: limit lower=-1.0472 upper=2.0944 effort=25 velocity=37 -> lower=-0.7 upper=2.0944 effort=25 velocity=37
- joint right_shoulder_pitch_joint: limit lower=-3.0892 upper=2.6704 effort=25 velocity=37 -> lower=-1.3 upper=1.3 effort=25 velocity=37
- joint right_shoulder_roll_joint: limit lower=-2.2515 upper=1.5882 effort=25 velocity=37 -> lower=-1.59 upper=-0.1 effort=25 velocity=37

Commit message: should yaw joint limits updated to sane values

File: assets/g1/g1_29dof_with_hand_rev_1_0.urdf (robot description, URDF)
Before this commit: robot g1_29dof_with_hand_rev_1_0, 54 links, 53 joints
Joints:
- joint left_shoulder_yaw_joint: limit lower=-2.618 upper=2.618 effort=25 velocity=37 -> lower=-0.2 upper=1.3 effort=25 velocity=37
- joint right_shoulder_yaw_joint: limit lower=-2.618 upper=2.618 effort=25 velocity=37 -> lower=-1.3 upper=0.2 effort=25 velocity=37

Commit message: relaxed joint limits

File: assets/g1/g1_29dof_with_hand_rev_1_0.urdf (robot description, URDF)
Before this commit: robot g1_29dof_with_hand_rev_1_0, 54 links, 53 joints
Joints:
- joint left_shoulder_roll_joint: limit lower=0.1 upper=1.59 effort=25 velocity=37 -> lower=0.01 upper=1.59 effort=25 velocity=37
- joint left_shoulder_yaw_joint: limit lower=-0.2 upper=1.3 effort=25 velocity=37 -> lower=-0.4 upper=1.3 effort=25 velocity=37
- joint right_shoulder_roll_joint: limit lower=-1.59 upper=-0.1 effort=25 velocity=37 -> lower=-1.59 upper=-0.01 effort=25 velocity=37
- joint right_shoulder_yaw_joint: limit lower=-1.3 upper=0.2 effort=25 velocity=37 -> lower=-1.3 upper=0.4 effort=25 velocity=37

Commit message: relaxing joint limits

File: assets/g1/g1_29dof_with_hand_rev_1_0.urdf (robot description, URDF)
Before this commit: robot g1_29dof_with_hand_rev_1_0, 54 links, 53 joints
Joints:
- joint left_elbow_joint: limit lower=-0.7 upper=2.0944 effort=25 velocity=37 -> lower=-1.0 upper=2.0944 effort=25 velocity=37
- joint right_elbow_joint: limit lower=-0.7 upper=2.0944 effort=25 velocity=37 -> lower=-1.0 upper=2.0944 effort=25 velocity=37
