Commit message: moving assets and viz to a new dependency free package

File: g1_description/assets/g1/g1_29dof_with_hand_rev_1_0_ros.urdf (robot description, URDF)
Before this commit: robot g1_29dof_with_hand_rev_1_0, 54 links, 53 joints
Links:
- link head_link: geometry collision mesh filename=package://g1_description/assets/g1/meshes/head_link.STL; visual mesh filename=package://g1_description/assets/g1/meshes/head_link.STL
- link left_ankle_pitch_link: geometry collision mesh filename=package://g1_description/assets/g1/meshes/left_ankle_pitch_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; visual mesh filename=package://g1_description/assets/g1/meshes/left_ankle_pitch_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
- link left_ankle_roll_link: geometry collision sphere radius=0.005; collision sphere radius=0.005
- link left_elbow_link: geometry collision mesh filename=package://g1_description/assets/g1/meshes/left_elbow_link.S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; visual mesh filename=package://g1_description/assets/g1/meshes/left_elbow_link.S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
- link left_hand_index_0_link: geometry collision mesh filename=package://g1_description/assets/g1/meshes/left_hand_index_0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; visual mesh filename=package://g1_description/assets/g1/meshes/left_hand_index_0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
- link left_hand_index_1_link: geometry collision mesh filename=package://g1_description/assets/g1/meshes/left_hand_index_1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; visual mesh filename=package://g1_description/assets/g1/meshes/left_hand_index_1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
- link left_hand_middle_0_link: geometry collision mesh filename=package://g1_description/assets/g1/meshes/left_hand_middle_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; visual mesh filename=package://g1_description/assets/g1/meshes/left_hand_middle_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
- link left_hand_middle_1_link: geometry collision mesh filename=package://g1_description/assets/g1/meshes/left_hand_middle_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; visual mesh filename=package://g1_description/assets/g1/meshes/left_hand_middle_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
- link left_hand_palm_link: geometry collision mesh filename=package://g1_description/assets/g1/meshes/left_hand_palm_li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; visual mesh filename=package://g1_description/assets/g1/meshes/left_hand_palm_li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
- link left_hand_thumb_0_link: geometry collision mesh filename=package://g1_description/assets/g1/meshes/left_hand_thumb_0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; visual mesh filename=package://g1_description/assets/g1/meshes/left_hand_thumb_0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
- link left_hand_thumb_1_link: geometry collision box size=0.02 0.03 0.02; visual mesh filename=package://g1_description/assets/g1/meshes/left_hand_thumb_1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
- link left_hand_thumb_2_link: geometry collision mesh filename=package://g1_description/assets/g1/meshes/left_hand_thumb_2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; visual mesh filename=package://g1_description/assets/g1/meshes/left_hand_thumb_2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
- link left_hip_pitch_link: geometry collision mesh filename=package://g1_description/assets/g1/meshes/left_hip_pitch_li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; visual mesh filename=package://g1_description/assets/g1/meshes/left_hip_pitch_li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
- link left_hip_roll_link: geometry collision mesh filename=package://g1_description/assets/g1/meshes/left_hip_roll_lin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; visual mesh filename=package://g1_description/assets/g1/meshes/left_hip_roll_lin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
- link left_hip_yaw_link: geometry collision mesh filename=package://g1_description/assets/g1/meshes/left_hip_yaw_link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; visual mesh filename=package://g1_description/assets/g1/meshes/left_hip_yaw_link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
- link left_knee_link: geometry collision mesh filename=package://g1_description/assets/g1/meshes/left_knee_link.STL; visual mesh filename=package://g1_description/assets/g1/meshes/left_knee_link.STL
- link left_shoulder_pitch_link: geometry collision cylinder length=0.05 radius=0.03; visual mesh filename=package://g1_description/assets/g1/meshes/left_shoulder_pit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
- link left_shoulder_roll_link: geometry collision cylinder length=0.03 radius=0.03; visual mesh filename=package://g1_description/assets/g1/meshes/left_shoulder_rol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
- link left_shoulder_yaw_link: geometry collision mesh filename=package://g1_description/assets/g1/meshes/left_shoulder_yaw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; visual mesh filename=package://g1_description/assets/g1/meshes/left_shoulder_yaw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
- link left_wrist_pitch_link: geometry collision mesh filename=package://g1_description/assets/g1/meshes/left_wrist_pitch_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; visual mesh filename=package://g1_description/assets/g1/meshes/left_wrist_pitch_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
- link left_wrist_roll_link: geometry collision mesh filename=package://g1_description/assets/g1/meshes/left_wrist_roll_l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; visual mesh filename=package://g1_description/assets/g1/meshes/left_wrist_roll_l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
- link left_wrist_yaw_link: geometry collision mesh filename=package://g1_description/assets/g1/meshes/left_wrist_yaw_li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; visual mesh filename=package://g1_description/assets/g1/meshes/left_wrist_yaw_li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
- link logo_link: geometry collision mesh filename=package://g1_description/assets/g1/meshes/logo_link.STL; visual mesh filename=package://g1_description/assets/g1/meshes/logo_link.STL
- link pelvis: geometry visual mesh filename=package://g1_description/assets/g1/meshes/pelvis.STL
- link pelvis_contour_link: geometry collision mesh filename=package://g1_description/assets/g1/meshes/pelvis_contour_li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; visual mesh filename=package://g1_description/assets/g1/meshes/pelvis_contour_li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
- link right_ankle_pitch_link: geometry collision mesh filename=package://g1_description/assets/g1/meshes/right_ankle_pitch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; visual mesh filename=package://g1_description/assets/g1/meshes/right_ankle_pitch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
- link right_ankle_roll_link: geometry collision sphere radius=0.005; collision sphere radius=0.005
- link right_elbow_link: geometry collision mesh filename=package://g1_description/assets/g1/meshes/right_elbow_link.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; visual mesh filename=package://g1_description/assets/g1/meshes/right_elbow_link.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
- link right_hand_index_0_link: geometry collision mesh filename=package://g1_description/assets/g1/meshes/right_hand_index_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; visual mesh filename=package://g1_description/assets/g1/meshes/right_hand_index_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
- link right_hand_index_1_link: geometry collision mesh filename=package://g1_description/assets/g1/meshes/right_hand_index_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; visual mesh filename=package://g1_description/assets/g1/meshes/right_hand_index_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
- link right_hand_middle_0_link: geometry collision mesh filename=package://g1_description/assets/g1/meshes/right_hand_middle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; visual mesh filename=package://g1_description/assets/g1/meshes/right_hand_middle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
- link right_hand_middle_1_link: geometry collision mesh filename=package://g1_description/assets/g1/meshes/right_hand_middle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; visual mesh filename=package://g1_description/assets/g1/meshes/right_hand_middle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
- link right_hand_palm_link: geometry collision mesh filename=package://g1_description/assets/g1/meshes/right_hand_palm_l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; visual mesh filename=package://g1_description/assets/g1/meshes/right_hand_palm_l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
- link right_hand_thumb_0_link: geometry collision mesh filename=package://g1_description/assets/g1/meshes/right_hand_thumb_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; visual mesh filename=package://g1_description/assets/g1/meshes/right_hand_thumb_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
- link right_hand_thumb_1_link: geometry collision box size=0.02 0.03 0.02; visual mesh filename=package://g1_description/assets/g1/meshes/right_hand_thumb_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
- link right_hand_thumb_2_link: geometry collision mesh filename=package://g1_description/assets/g1/meshes/right_hand_thumb_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; visual mesh filename=package://g1_description/assets/g1/meshes/right_hand_thumb_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
- link right_hip_pitch_link: geometry collision mesh filename=package://g1_description/assets/g1/meshes/right_hip_pitch_l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; visual mesh filename=package://g1_description/assets/g1/meshes/right_hip_pitch_l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
- link right_hip_roll_link: geometry collision mesh filename=package://g1_description/assets/g1/meshes/right_hip_roll_li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; visual mesh filename=package://g1_description/assets/g1/meshes/right_hip_roll_li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
- link right_hip_yaw_link: geometry collision mesh filename=package://g1_description/assets/g1/meshes/right_hip_yaw_lin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; visual mesh filename=package://g1_description/assets/g1/meshes/right_hip_yaw_lin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
- link right_knee_link: geometry collision mesh filename=package://g1_description/assets/g1/meshes/right_knee_link.S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; visual mesh filename=package://g1_description/assets/g1/meshes/right_knee_link.S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
- link right_shoulder_pitch_link: geometry collision cylinder length=0.05 radius=0.03; visual mesh filename=package://g1_description/assets/g1/meshes/right_shoulder_pi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
- link right_shoulder_roll_link: geometry collision cylinder length=0.03 radius=0.03; visual mesh filename=package://g1_description/assets/g1/meshes/right_shoulder_ro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
- link right_shoulder_yaw_link: geometry collision mesh filename=package://g1_description/assets/g1/meshes/right_shoulder_ya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; visual mesh filename=package://g1_description/assets/g1/meshes/right_shoulder_ya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
- link right_wrist_pitch_link: geometry collision mesh filename=package://g1_description/assets/g1/meshes/right_wrist_pitch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; visual mesh filename=package://g1_description/assets/g1/meshes/right_wrist_pitch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
- link right_wrist_roll_link: geometry collision mesh filename=package://g1_description/assets/g1/meshes/right_wrist_roll_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; visual mesh filename=package://g1_description/assets/g1/meshes/right_wrist_roll_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
- link right_wrist_yaw_link: geometry collision mesh filename=package://g1_description/assets/g1/meshes/right_wrist_yaw_l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; visual mesh filename=package://g1_description/assets/g1/meshes/right_wrist_yaw_l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
- link torso_link: geometry collision mesh filename=package://g1_description/assets/g1/meshes/torso_link_rev_1_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; visual mesh filename=package://g1_description/assets/g1/meshes/torso_link_rev_1_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
- link waist_roll_link: geometry visual mesh filename=package://g1_description/assets/g1/meshes/waist_roll_link_r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
- link waist_yaw_link: geometry visual mesh filename=package://g1_description/assets/g1/meshes/waist_yaw_link_re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
Joints:
- joint d435_joint: origin xyz=0.0856235 0.03553 0.4407 rpy=0 0.501426 0 -> xyz=0.068042 0.016300 0.414516 rpy=-0.011720 0.453641 0.026073
- joint g1_reference_to_pelvis_joint: child pelvis -> base_link; parent base_link -> pelvis
- joint mid360_joint: child sensor -> torso_link; origin xyz=0.0002835 0.00003 0.41618 rpy=0 0.04014257279586953 0 -> xyz=-0.0002835 -0.00003 -0.41618 rpy=0 -0.04014257279586953 0; parent torso_link -> sensor
- joint waist_pitch_joint: axis 0 1 0 -> 0 -1 0; child torso_link -> waist_roll_link; parent waist_roll_link -> torso_link
- joint waist_roll_joint: axis 1 0 0 -> -1 0 0; child waist_roll_link -> waist_yaw_link; origin xyz=-0.0039635 0 0.044 rpy=0 0 0 -> xyz=0.0039635 0 -0.044 rpy=0 0 0; parent waist_yaw_link -> waist_roll_link
- joint waist_yaw_joint: axis 0 0 1 -> 0 0 -1; child waist_yaw_link -> pelvis; parent pelvis -> waist_yaw_link

File: g1_description/assets/g1/g1_29dof_with_hand_rev_1_0_ros_ctrl_viz.urdf (robot description, URDF)
Before this commit: robot g1_29dof_with_hand_rev_1_0, 54 links, 53 joints
Links:
- link head_link: geometry collision mesh filename=package://g1_description/assets/g1/meshes/head_link.STL; visual mesh filename=package://g1_description/assets/g1/meshes/head_link.STL
- link left_ankle_pitch_link: geometry collision mesh filename=package://g1_description/assets/g1/meshes/left_ankle_pitch_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; visual mesh filename=package://g1_description/assets/g1/meshes/left_ankle_pitch_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
- link left_ankle_roll_link: geometry collision sphere radius=0.005; collision sphere radius=0.005
- link left_elbow_link: geometry collision mesh filename=package://g1_description/assets/g1/meshes/left_elbow_link.S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; visual mesh filename=package://g1_description/assets/g1/meshes/left_elbow_link.S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
- link left_hand_index_0_link: geometry collision mesh filename=package://g1_description/assets/g1/meshes/left_hand_index_0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; visual mesh filename=package://g1_description/assets/g1/meshes/left_hand_index_0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
- link left_hand_index_1_link: geometry collision mesh filename=package://g1_description/assets/g1/meshes/left_hand_index_1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; visual mesh filename=package://g1_description/assets/g1/meshes/left_hand_index_1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
- link left_hand_middle_0_link: geometry collision mesh filename=package://g1_description/assets/g1/meshes/left_hand_middle_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; visual mesh filename=package://g1_description/assets/g1/meshes/left_hand_middle_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
- link left_hand_middle_1_link: geometry collision mesh filename=package://g1_description/assets/g1/meshes/left_hand_middle_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; visual mesh filename=package://g1_description/assets/g1/meshes/left_hand_middle_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
- link left_hand_palm_link: geometry collision mesh filename=package://g1_description/assets/g1/meshes/left_hand_palm_li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; visual mesh filename=package://g1_description/assets/g1/meshes/left_hand_palm_li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
- link left_hand_thumb_0_link: geometry collision mesh filename=package://g1_description/assets/g1/meshes/left_hand_thumb_0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; visual mesh filename=package://g1_description/assets/g1/meshes/left_hand_thumb_0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
- link left_hand_thumb_1_link: geometry collision box size=0.02 0.03 0.02; visual mesh filename=package://g1_description/assets/g1/meshes/left_hand_thumb_1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
- link left_hand_thumb_2_link: geometry collision mesh filename=package://g1_description/assets/g1/meshes/left_hand_thumb_2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; visual mesh filename=package://g1_description/assets/g1/meshes/left_hand_thumb_2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
- link left_hip_pitch_link: geometry collision mesh filename=package://g1_description/assets/g1/meshes/left_hip_pitch_li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; visual mesh filename=package://g1_description/assets/g1/meshes/left_hip_pitch_li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
- link left_hip_roll_link: geometry collision mesh filename=package://g1_description/assets/g1/meshes/left_hip_roll_lin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; visual mesh filename=package://g1_description/assets/g1/meshes/left_hip_roll_lin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
- link left_hip_yaw_link: geometry collision mesh filename=package://g1_description/assets/g1/meshes/left_hip_yaw_link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; visual mesh filename=package://g1_description/assets/g1/meshes/left_hip_yaw_link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
- link left_knee_link: geometry collision mesh filename=package://g1_description/assets/g1/meshes/left_knee_link.STL; visual mesh filename=package://g1_description/assets/g1/meshes/left_knee_link.STL
- link left_shoulder_pitch_link: geometry collision cylinder length=0.05 radius=0.03; visual mesh filename=package://g1_description/assets/g1/meshes/left_shoulder_pit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
- link left_shoulder_roll_link: geometry collision cylinder length=0.03 radius=0.03; visual mesh filename=package://g1_description/assets/g1/meshes/left_shoulder_rol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
- link left_shoulder_yaw_link: geometry collision mesh filename=package://g1_description/assets/g1/meshes/left_shoulder_yaw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; visual mesh filename=package://g1_description/assets/g1/meshes/left_shoulder_yaw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
- link left_wrist_pitch_link: geometry collision mesh filename=package://g1_description/assets/g1/meshes/left_wrist_pitch_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; visual mesh filename=package://g1_description/assets/g1/meshes/left_wrist_pitch_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
- link left_wrist_roll_link: geometry collision mesh filename=package://g1_description/assets/g1/meshes/left_wrist_roll_l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; visual mesh filename=package://g1_description/assets/g1/meshes/left_wrist_roll_l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
- link left_wrist_yaw_link: geometry collision mesh filename=package://g1_description/assets/g1/meshes/left_wrist_yaw_li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; visual mesh filename=package://g1_description/assets/g1/meshes/left_wrist_yaw_li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
- link logo_link: geometry collision mesh filename=package://g1_description/assets/g1/meshes/logo_link.STL; visual mesh filename=package://g1_description/assets/g1/meshes/logo_link.STL
- link pelvis: geometry visual mesh filename=package://g1_description/assets/g1/meshes/pelvis.STL
- link pelvis_contour_link: geometry collision mesh filename=package://g1_description/assets/g1/meshes/pelvis_contour_li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; visual mesh filename=package://g1_description/assets/g1/meshes/pelvis_contour_li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
- link right_ankle_pitch_link: geometry collision mesh filename=package://g1_description/assets/g1/meshes/right_ankle_pitch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; visual mesh filename=package://g1_description/assets/g1/meshes/right_ankle_pitch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
- link right_ankle_roll_link: geometry collision sphere radius=0.005; collision sphere radius=0.005
- link right_elbow_link: geometry collision mesh filename=package://g1_description/assets/g1/meshes/right_elbow_link.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; visual mesh filename=package://g1_description/assets/g1/meshes/right_elbow_link.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
- link right_hand_index_0_link: geometry collision mesh filename=package://g1_description/assets/g1/meshes/right_hand_index_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; visual mesh filename=package://g1_description/assets/g1/meshes/right_hand_index_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
- link right_hand_index_1_link: geometry collision mesh filename=package://g1_description/assets/g1/meshes/right_hand_index_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; visual mesh filename=package://g1_description/assets/g1/meshes/right_hand_index_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
- link right_hand_middle_0_link: geometry collision mesh filename=package://g1_description/assets/g1/meshes/right_hand_middle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; visual mesh filename=package://g1_description/assets/g1/meshes/right_hand_middle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
- link right_hand_middle_1_link: geometry collision mesh filename=package://g1_description/assets/g1/meshes/right_hand_middle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; visual mesh filename=package://g1_description/assets/g1/meshes/right_hand_middle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
- link right_hand_palm_link: geometry collision mesh filename=package://g1_description/assets/g1/meshes/right_hand_palm_l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; visual mesh filename=package://g1_description/assets/g1/meshes/right_hand_palm_l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
- link right_hand_thumb_0_link: geometry collision mesh filename=package://g1_description/assets/g1/meshes/right_hand_thumb_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; visual mesh filename=package://g1_description/assets/g1/meshes/right_hand_thumb_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
- link right_hand_thumb_1_link: geometry collision box size=0.02 0.03 0.02; visual mesh filename=package://g1_description/assets/g1/meshes/right_hand_thumb_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
- link right_hand_thumb_2_link: geometry collision mesh filename=package://g1_description/assets/g1/meshes/right_hand_thumb_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; visual mesh filename=package://g1_description/assets/g1/meshes/right_hand_thumb_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
- link right_hip_pitch_link: geometry collision mesh filename=package://g1_description/assets/g1/meshes/right_hip_pitch_l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; visual mesh filename=package://g1_description/assets/g1/meshes/right_hip_pitch_l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
- link right_hip_roll_link: geometry collision mesh filename=package://g1_description/assets/g1/meshes/right_hip_roll_li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; visual mesh filename=package://g1_description/assets/g1/meshes/right_hip_roll_li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
- link right_hip_yaw_link: geometry collision mesh filename=package://g1_description/assets/g1/meshes/right_hip_yaw_lin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; visual mesh filename=package://g1_description/assets/g1/meshes/right_hip_yaw_lin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
- link right_knee_link: geometry collision mesh filename=package://g1_description/assets/g1/meshes/right_knee_link.S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; visual mesh filename=package://g1_description/assets/g1/meshes/right_knee_link.S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
- link right_shoulder_pitch_link: geometry collision cylinder length=0.05 radius=0.03; visual mesh filename=package://g1_description/assets/g1/meshes/right_shoulder_pi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
- link right_shoulder_roll_link: geometry collision cylinder length=0.03 radius=0.03; visual mesh filename=package://g1_description/assets/g1/meshes/right_shoulder_ro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
- link right_shoulder_yaw_link: geometry collision mesh filename=package://g1_description/assets/g1/meshes/right_shoulder_ya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; visual mesh filename=package://g1_description/assets/g1/meshes/right_shoulder_ya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
- link right_wrist_pitch_link: geometry collision mesh filename=package://g1_description/assets/g1/meshes/right_wrist_pitch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; visual mesh filename=package://g1_description/assets/g1/meshes/right_wrist_pitch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
- link right_wrist_roll_link: geometry collision mesh filename=package://g1_description/assets/g1/meshes/right_wrist_roll_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; visual mesh filename=package://g1_description/assets/g1/meshes/right_wrist_roll_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
- link right_wrist_yaw_link: geometry collision mesh filename=package://g1_description/assets/g1/meshes/right_wrist_yaw_l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; visual mesh filename=package://g1_description/assets/g1/meshes/right_wrist_yaw_l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
- link torso_link: geometry collision mesh filename=package://g1_description/assets/g1/meshes/torso_link_rev_1_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; visual mesh filename=package://g1_description/assets/g1/meshes/torso_link_rev_1_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
- link waist_roll_link: geometry visual mesh filename=package://g1_description/assets/g1/meshes/waist_roll_link_r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
- link waist_yaw_link: geometry visual mesh filename=package://g1_description/assets/g1/meshes/waist_yaw_link_re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
Joints:
- joint d435_joint: origin xyz=0.068042 0.016300 0.414516 rpy=-0.011720 0.453641 0.026073 -> xyz=0.0856235 0.03553 0.4407 rpy=0 0.501426 0
- joint g1_reference_to_pelvis_joint: child base_link -> pelvis; parent pelvis -> base_link
- joint mid360_joint: child torso_link -> sensor; origin xyz=-0.0002835 -0.00003 -0.41618 rpy=0 -0.04014257279586953 0 -> xyz=0.0002835 0.00003 0.41618 rpy=0 0.04014257279586953 0; parent sensor -> torso_link
- joint waist_pitch_joint: axis 0 -1 0 -> 0 1 0; child waist_roll_link -> torso_link; parent torso_link -> waist_roll_link
- joint waist_roll_joint: axis -1 0 0 -> 1 0 0; child waist_yaw_link -> waist_roll_link; origin xyz=0.0039635 0 -0.044 rpy=0 0 0 -> xyz=-0.0039635 0 0.044 rpy=0 0 0; parent waist_roll_link -> waist_yaw_link
- joint waist_yaw_joint: axis 0 0 -1 -> 0 0 1; child pelvis -> waist_yaw_link; parent waist_yaw_link -> pelvis
