Commit message: moving custom joint limits to config

File: g1_description/assets/g1/g1_29dof_with_hand_rev_1_0.urdf (robot description, URDF)
Before this commit: robot g1_29dof_with_hand_rev_1_0, 54 links, 53 joints
Joints:
- joint d435_joint: origin xyz=0.0799335 0.01753 0.41036 rpy=0 0.401426 0 -> xyz=0.0576235 0.01753 0.42987 rpy=0 0.8308 0
- joint left_elbow_joint: limit lower=-1.0 upper=2.0944 effort=25 velocity=37 -> lower=-1.0472 upper=2.0944 effort=25 velocity=37
- joint left_shoulder_pitch_joint: limit lower=-1.3 upper=1.3 effort=25 velocity=37 -> lower=-3.0892 upper=2.6704 effort=25 velocity=37
- joint left_shoulder_roll_joint: limit lower=0.01 upper=1.59 effort=25 velocity=37 -> lower=-1.5882 upper=2.2515 effort=25 velocity=37
- joint left_shoulder_yaw_joint: limit lower=-0.4 upper=1.3 effort=25 velocity=37 -> lower=-2.618 upper=2.618 effort=25 velocity=37
- joint right_elbow_joint: limit lower=-1.0 upper=2.0944 effort=25 velocity=37 -> lower=-1.0472 upper=2.0944 effort=25 velocity=37
- joint right_shoulder_pitch_joint: limit lower=-1.3 upper=1.3 effort=25 velocity=37 -> lower=-3.0892 upper=2.6704 effort=25 velocity=37
- joint right_shoulder_roll_joint: limit lower=-1.59 upper=-0.01 effort=25 velocity=37 -> lower=-2.2515 upper=1.5882 effort=25 velocity=37
- joint right_shoulder_yaw_joint: limit lower=-1.3 upper=0.4 effort=25 velocity=37 -> lower=-2.618 upper=2.618 effort=25 velocity=37
